Commit message: complete, but lack of hw to run

File: src/main_bot/description/lidar.xacro (robot description, xacro)
@@ -30,7 +30,11 @@
     <gazebo reference="lidar_frame">
         <sensor name="lidar" type="gpu_lidar">
+            <!-- gz_frame_id stays unprefixed: robot_state_publisher isn't renaming
+                 URDF link names, it just gets its own /<robot_name>/tf topic via
+                 node namespacing, so "lidar_frame" is still the frame it publishes
+                 there. Only the gz-transport topic needs a unique name per robot. -->
             <gz_frame_id>lidar_frame</gz_frame_id>
             <pose>0 0 0 0 0 0</pose>
-            <topic>scan</topic>
+            <topic>${frame_prefix}scan</topic>
             <update_rate>10</update_rate>
             <always_on>1</always_on>
@@ -62,8 +66,8 @@
                 </noise>
             </lidar>
-        <plugin filename="gz-sim-sensors-system"
-                name="gz::sim::systems::Sensors">
-                <render_engine>ogre2</render_engine>
-        </plugin>
+        <!-- The Sensors system plugin is declared once at the world level
+             (worlds/warehouse.sdf) instead of per-robot here: it's a world-level
+             singleton, and re-registering it for a second spawned robot raced
+             and crashed the renderer. -->
         </sensor>
     </gazebo>

File: src/main_bot/description/robot.urdf.xacro (robot description, xacro)
@@ -1,8 +1,27 @@
 <?xml version="1.0"?>
 <robot xmlns:xacro="http://www.ros.org/wiki/xacro"  name="robot">
+    <!-- Multi-robot support: empty by default so single-robot launches
+         (gz.launch.py, slam.launch.py, nav2.launch.py) are unaffected.
+         Pass robot_name (no slash, e.g. "robot1") to get a ROS namespace
+         for the controller_manager and a "robot1/" tf/topic prefix. -->
+    <xacro:arg name="robot_name" default=""/>
+    <xacro:property name="robot_name" value="$(arg robot_name)"/>
+    <xacro:property name="frame_prefix" value="${'' if robot_name == '' else robot_name + '/'}"/>
+    <!-- ros2_control (via gz_ros2_control) is the default: it's what gz.launch.py /
+         slam.launch.py / nav2.launch.py are built and tested against for a single
+         robot. gz_ros2_control has proven unreliable running multiple controller_manager
+         instances in one Gazebo process, so multi_robot.launch.py sets this false to
+         get the plain gz-sim DiffDrive plugin instead (no per-robot controller_manager). -->
+    <xacro:arg name="use_ros2_control" default="true"/>
+    <xacro:property name="use_ros2_control" value="$(arg use_ros2_control)"/>
     <!-- Robot_frames -->
     <xacro:include filename = "robot_main.xacro" />
-    <!-- Controls (ros2_control via gz_ros2_control, Gazebo simulation) -->
-    <xacro:include filename = "ros2_controller.xacro" />
+    <!-- Controls -->
+    <xacro:if value="${use_ros2_control}">
+        <xacro:include filename = "ros2_controller.xacro" />
+    </xacro:if>
+    <xacro:unless value="${use_ros2_control}">
+        <xacro:include filename = "gz_diff_drive.xacro" />
+    </xacro:unless>
     <!-- Sensors -->
     <xacro:include filename = "lidar.xacro" />

File: src/main_bot/description/robot_main.xacro (robot description, xacro)
@@ -74,5 +74,8 @@
     </link>
     <gazebo reference="chasis">
-        <material>Gazebo/Blue</material>
+        <material>
+            <ambient>0 0 1 1</ambient>
+            <diffuse>0 0 1 1</diffuse>
+        </material>
     </gazebo>
     <!-- left_wheel -->
@@ -100,5 +103,8 @@
     </link>
     <gazebo reference="left_wheel">
-        <material>Gazebo/Black</material>
+        <material>
+            <ambient>0 0 0 1</ambient>
+            <diffuse>0 0 0 1</diffuse>
+        </material>
     </gazebo>
     <!-- right_wheel -->
@@ -126,5 +132,8 @@
     </link>
     <gazebo reference="right_wheel">
-        <material>Gazebo/Black</material>
+        <material>
+            <ambient>0 0 0 1</ambient>
+            <diffuse>0 0 0 1</diffuse>
+        </material>
     </gazebo>
     <!-- caster_wheel_front -->
@@ -151,5 +160,8 @@
     </link>
     <gazebo reference="caster_wheel_front">
-        <material>Gazebo/Orange</material>
+        <material>
+            <ambient>1 0.25 0 1</ambient>
+            <diffuse>1 0.25 0 1</diffuse>
+        </material>
         <mu1 value= "0.0001"/>
         <mu2 value= "0.0001"/>
@@ -178,5 +190,8 @@
     </link>
     <gazebo reference="caster_wheel_rear">
-        <material>Gazebo/Orange</material>
+        <material>
+            <ambient>1 0.25 0 1</ambient>
+            <diffuse>1 0.25 0 1</diffuse>
+        </material>
         <mu1 value= "0.0001"/>
         <mu2 value= "0.0001"/>

File: src/main_bot/description/ros2_controller.xacro (robot description, xacro)
@@ -26,4 +26,7 @@
                 name="gz_ros2_control::GazeboSimROS2ControlPlugin">
             <parameters>$(find main_bot)/config/controllers.yaml</parameters>
+            <ros>
+                <namespace>${robot_name}</namespace>
+            </ros>
         </plugin>
     </gazebo>
